File: generics/cap_0603.kicad_sch (KiCad schematic)
At the start: 7 parts

Commit message: - Add Schottky diode and rectifier bridge - Add generics
Parts:
- added C9: 4.7nF, Capacitor_SMD:C_0603_1608Metric, symbol Device:C_Small
- C21: Tolerance (none) -> 10%; Voltage (none) -> 25V
- C5: value 4.7nF -> 47nF
